Commit message: modelled the grabber

File: ros2_ws/src/rover_description/urdf/rover.urdf.xacro (robot description, xacro)
@@ -3,5 +3,5 @@
   <!-- load global parameters -->
   <xacro:property name="config_path" value="$(find rover_description)/config/physical_params.yaml" />
-  <xacro:property name="params" value="${xacro.load_yaml(config_path)}['robot_dimensions']" />
+  <xacro:property name="params" value="${xacro.load_yaml(config_path)['robot_dimensions']}" />
   <!-- extract values -->
   <xacro:property name="c_off" value="${params['column_base_offset']}" />
@@ -12,9 +12,31 @@
   <material name="black"><color rgba="0 0 0 1"/></material>
   <material name="blue"><color rgba="0 0 0.8 1"/></material>
-  <material name="red"><color rgba="0 0.8 0 1"/></material>
+  <material name="red"><color rgba="0.8 0 0 1"/></material>
   <material name="green"><color rgba="0 0.8 0 1"/></material>
   <link name="base_link">
     <visual><geometry><box size="4.0 4.0 1.0"/></geometry><material name="black"/></visual>
   </link>
+  <!-- define wheel macro -->
+  <xacro:macro name="wheel" params="prefix x_offset y_offset">
+    <joint name="${prefix}_wheel_joint" type="continuous">
+      <parent link="base_link"/>
+      <child link="${prefix}_wheel_link"/>
+      <origin xyz="${x_offset} ${y_offset} -0.3" rpy="0 0 0"/>
+      <axis xyz="0 1 0"/>
+    </joint>
+    <link name="${prefix}_wheel_link">
+      <visual>
+        <origin xyz="0 0 0" rpy="1.57079632679 0 0"/>
+        <geometry>
+          <cylinder radius="0.8" length="0.4"/>
+        </geometry>
+        <material name="black"/>
+      </visual>
+    </link>
+  </xacro:macro>
+  <xacro:wheel prefix="front_left" x_offset="1.5" y_offset="2.2"/>
+  <xacro:wheel prefix="front_right" x_offset="1.5" y_offset="-2.2"/>
+  <xacro:wheel prefix="rear_left" x_offset="-1.5" y_offset="2.2"/>
+  <xacro:wheel prefix="rear_right" x_offset="-1.5" y_offset="-2.2"/>
   <joint name="stand_column_joint" type="fixed">
     <parent link="base_link"/><child link="column_link"/>
@@ -46,3 +68,60 @@
     <visual><origin xyz="${t_len/2} 0 0"/><geometry><sphere radius="0.3"/></geometry><material name="green"/></visual>
   </link>
+  <!-- grabber / gripper fingers -->
+  <joint name="left_finger_joint" type="prismatic">
+    <parent link="tool_link"/><child link="left_finger_link"/>
+    <origin xyz="0.3 0.3 0" rpy="0 0 0"/>
+    <axis xyz="0 1 0"/>
+    <limit lower="-0.2" upper="0.2" effort="10" velocity="0.5"/>
+  </joint>
+  <link name="left_finger_link">
+    <visual><origin xyz="0.3 0 0"/><geometry><box size="0.6 0.1 0.3"/></geometry><material name="blue"/></visual>
+  </link>
+  <joint name="right_finger_joint" type="prismatic">
+    <parent link="tool_link"/><child link="right_finger_link"/>
+    <origin xyz="0.3 -0.3 0" rpy="0 0 0"/>
+    <axis xyz="0 -1 0"/>
+    <limit lower="-0.2" upper="0.2" effort="10" velocity="0.5"/>
+  </joint>
+  <link name="right_finger_link">
+    <visual><origin xyz="0.3 0 0"/><geometry><box size="0.6 0.1 0.3"/></geometry><material name="blue"/></visual>
+  </link>
+  <joint name="gripper_motor_body_joint" type="fixed">
+    <parent link="tool_link"/>
+    <child link="gripper_motor_body_link"/>
+    <origin xyz="0.3 0 0.35" rpy="0 0 0"/>
+  </joint>
+  <link name="gripper_motor_body_link">
+    <visual>
+      <geometry>
+        <box size="0.3 0.3 0.3"/>
+      </geometry>
+      <material name="black"/>
+    </visual>
+  </link>
+  <!-- i don't know the exact mechanism but this works now for simulations-->
+  <!-- stepper motor rotating shaft / lead screw (rotates around Y axis) -->
+  <joint name="gripper_motor_shaft_joint" type="continuous">
+    <parent link="gripper_motor_body_link"/>
+    <child link="gripper_motor_shaft_link"/>
+    <origin xyz="0 0 -0.2" rpy="0 0 0"/>
+    <axis xyz="0 1 0"/>
+  </joint>
+  <link name="gripper_motor_shaft_link">
+    <!-- main shaft cylinder -->
+    <visual>
+      <origin xyz="0 0 0" rpy="1.57079632679 0 0"/>
+      <geometry>
+        <cylinder radius="0.04" length="0.8"/>
+      </geometry>
+      <material name="red"/>
+    </visual>
+    <visual>
+      <origin xyz="0 0 0.05" rpy="0 0 0"/>
+      <geometry>
+        <box size="0.2 0.08 0.04"/>
+      </geometry>
+      <material name="red"/>
+    </visual>
+  </link>
 </robot>
